Commit message: fix(tianyi2): refine hand skeleton proportions

File: x-humanoid/tianyi2.0/resource/tianyi2_model.urdf (robot description, URDF)
Before this commit: robot Tianyi2Pro, 62 links, 61 joints
Joints:
- joint left_hand_index_tip: origin xyz=0 0 -0.070 rpy=0 0 0 -> xyz=0 0 -0.035 rpy=0 0 0
- joint left_hand_little_tip: origin xyz=0 0 -0.060 rpy=0 0 0 -> xyz=0 0 -0.030 rpy=0 0 0
- joint left_hand_middle_tip: origin xyz=0 0 -0.075 rpy=0 0 0 -> xyz=0 0 -0.0375 rpy=0 0 0
- joint left_hand_ring_tip: origin xyz=0 0 -0.070 rpy=0 0 0 -> xyz=0 0 -0.035 rpy=0 0 0
- joint left_hand_thumb_rotation_joint: origin xyz=0 0.035 -0.015 rpy=0 0 0 -> xyz=0 0.035 -0.015 rpy=0 0 -0.349066
- joint right_hand_index_tip: origin xyz=0 0 -0.070 rpy=0 0 0 -> xyz=0 0 -0.035 rpy=0 0 0
- joint right_hand_little_tip: origin xyz=0 0 -0.060 rpy=0 0 0 -> xyz=0 0 -0.030 rpy=0 0 0
- joint right_hand_middle_tip: origin xyz=0 0 -0.075 rpy=0 0 0 -> xyz=0 0 -0.0375 rpy=0 0 0
- joint right_hand_ring_tip: origin xyz=0 0 -0.070 rpy=0 0 0 -> xyz=0 0 -0.035 rpy=0 0 0
- joint right_hand_thumb_rotation_joint: origin xyz=0 -0.035 -0.015 rpy=0 0 0 -> xyz=0 -0.035 -0.015 rpy=0 0 0.349066

Commit message: fix(tianyi2): mirror right-hand finger order

File: x-humanoid/tianyi2.0/resource/tianyi2_model.urdf (robot description, URDF)
Before this commit: robot Tianyi2Pro, 62 links, 61 joints
Joints:
- joint right_hand_index_distal_joint: origin xyz=0 0 -0.035 rpy=0 0 0 -> xyz=0 0 -0.030 rpy=0 0 0
- joint right_hand_index_joint: origin xyz=0 0.015 -0.060 rpy=0 0 0 -> xyz=0 -0.03 -0.050 rpy=0 0 0
- joint right_hand_index_tip: origin xyz=0 0 -0.035 rpy=0 0 0 -> xyz=0 0 -0.030 rpy=0 0 0
- joint right_hand_little_distal_joint: origin xyz=0 0 -0.030 rpy=0 0 0 -> xyz=0 0 -0.035 rpy=0 0 0
- joint right_hand_little_joint: origin xyz=0 -0.03 -0.050 rpy=0 0 0 -> xyz=0 0.015 -0.060 rpy=0 0 0
- joint right_hand_little_tip: origin xyz=0 0 -0.030 rpy=0 0 0 -> xyz=0 0 -0.035 rpy=0 0 0
- joint right_hand_middle_distal_joint: origin xyz=0 0 -0.0375 rpy=0 0 0 -> xyz=0 0 -0.035 rpy=0 0 0
- joint right_hand_middle_joint: origin xyz=0 0 -0.0655 rpy=0 0 0 -> xyz=0 -0.015 -0.060 rpy=0 0 0
- joint right_hand_middle_tip: origin xyz=0 0 -0.0375 rpy=0 0 0 -> xyz=0 0 -0.035 rpy=0 0 0
- joint right_hand_ring_distal_joint: origin xyz=0 0 -0.035 rpy=0 0 0 -> xyz=0 0 -0.0375 rpy=0 0 0
- joint right_hand_ring_joint: origin xyz=0 -0.015 -0.060 rpy=0 0 0 -> xyz=0 0 -0.0655 rpy=0 0 0
- joint right_hand_ring_tip: origin xyz=0 0 -0.035 rpy=0 0 0 -> xyz=0 0 -0.0375 rpy=0 0 0

Commit message: fix(tianyi2): preserve right-hand finger geometry

File: x-humanoid/tianyi2.0/resource/tianyi2_model.urdf (robot description, URDF)
Before this commit: robot Tianyi2Pro, 62 links, 61 joints
Joints:
- joint right_hand_index_distal_joint: origin xyz=0 0 -0.030 rpy=0 0 0 -> xyz=0 0 -0.035 rpy=0 0 0
- joint right_hand_index_joint: origin xyz=0 -0.03 -0.050 rpy=0 0 0 -> xyz=0 -0.015 -0.060 rpy=0 0 0
- joint right_hand_index_tip: origin xyz=0 0 -0.030 rpy=0 0 0 -> xyz=0 0 -0.035 rpy=0 0 0
- joint right_hand_little_distal_joint: origin xyz=0 0 -0.035 rpy=0 0 0 -> xyz=0 0 -0.030 rpy=0 0 0
- joint right_hand_little_joint: origin xyz=0 0.015 -0.060 rpy=0 0 0 -> xyz=0 0.030 -0.050 rpy=0 0 0
- joint right_hand_little_tip: origin xyz=0 0 -0.035 rpy=0 0 0 -> xyz=0 0 -0.030 rpy=0 0 0
- joint right_hand_middle_distal_joint: origin xyz=0 0 -0.035 rpy=0 0 0 -> xyz=0 0 -0.0375 rpy=0 0 0
- joint right_hand_middle_joint: origin xyz=0 -0.015 -0.060 rpy=0 0 0 -> xyz=0 0 -0.0655 rpy=0 0 0
- joint right_hand_middle_tip: origin xyz=0 0 -0.035 rpy=0 0 0 -> xyz=0 0 -0.0375 rpy=0 0 0
- joint right_hand_ring_distal_joint: origin xyz=0 0 -0.0375 rpy=0 0 0 -> xyz=0 0 -0.035 rpy=0 0 0
- joint right_hand_ring_joint: origin xyz=0 0 -0.0655 rpy=0 0 0 -> xyz=0 0.015 -0.060 rpy=0 0 0
- joint right_hand_ring_tip: origin xyz=0 0 -0.0375 rpy=0 0 0 -> xyz=0 0 -0.035 rpy=0 0 0
